Commit message: Added mount part to urdf xacro

File: ur5_allegro.xacro (robot description, xacro)
@@ -1,5 +1,5 @@
 <?xml version="1.0"?>
 <!--- <robot xmlns:xacro="http://ros.org/wiki/xacro" name="ur5" >  -->
-<robot xmlns:xacro="http://www.ros.org/wiki/xacro" name="ur5" >
+<robot xmlns:xacro="http://ros.org/wiki/xacro" name="ur5_allegro" >
   <!-- allegro -->
   <xacro:include filename="$(find allegro_hand_description)/allegro_hand_description_right.xacro" />
@@ -8,4 +8,6 @@
   <!-- arm -->
   <xacro:ur5_robot prefix="" joint_limited="false"/>
+  <!-- mount part connecting allegro to ur5-->
+  <xacro:include filename="$(find ur5_allegro_moveit)/mount_part.xacro" />
   <link name="world" />
   <joint name="world_joint" type="fixed">
@@ -16,6 +18,11 @@
   <joint name="ee_mount" type="fixed">
     <parent link="ee_link" />
+    <child link = "mount_base" />
+    <origin xyz="0.0025 0.0 0.0" rpy="0.0 1.5708 0.0" />
+  </joint>
+  <joint name="mount_allegro" type="fixed">
+    <parent link="mount_body" />
     <child link = "hand_root" />
-    <origin xyz="0.0 0.0 0.0" rpy="0.0 1.5708 0.0" />
+    <origin xyz="0.0 0.0 0.0375" rpy="0.0 0.0 0.0" />
   </joint>
 </robot>

Commit message: Xacro base link orientation as on the real robot

File: ur5_allegro.xacro (robot description, xacro)
@@ -14,5 +14,5 @@
     <parent link="world" />
     <child link = "base_link" />
-    <origin xyz="0.0 0.0 0.0" rpy="0.0 0.0 0.0" />
+    <origin xyz="0.0 0.0 0.0" rpy="1.5708 0.0 1.5708" />
   </joint>
   <joint name="ee_mount" type="fixed">

Commit message: Xacro: Rotate hand

File: ur5_allegro.xacro (robot description, xacro)
@@ -24,5 +24,5 @@
     <parent link="mount_body" />
     <child link = "hand_root" />
-    <origin xyz="0.0 0.0 0.0375" rpy="0.0 0.0 0.0" />
+    <origin xyz="0.0 0.0 0.0375" rpy="0.0 0.0 2.356" />
   </joint>
 </robot>

Commit message: ur5_allegro xacro: joints between world ur5 and allegro

File: ur5_allegro.xacro (robot description, xacro)
@@ -13,9 +13,9 @@
   <joint name="world_joint" type="fixed">
     <parent link="world" />
-    <child link = "base_link" />
+    <child link = "base" />
     <origin xyz="0.0 0.0 0.0" rpy="1.5708 0.0 1.5708" />
   </joint>
-  <joint name="ee_mount" type="fixed">
-    <parent link="ee_link" />
+  <joint name="tool_mount" type="fixed">
+    <parent link="tool0" />
     <child link = "mount_base" />
     <origin xyz="0.0025 0.0 0.0" rpy="0.0 1.5708 0.0" />

Commit message: Re-generated package with new tool joint

File: ur5_allegro.xacro (robot description, xacro)
@@ -13,5 +13,5 @@
   <joint name="world_joint" type="fixed">
     <parent link="world" />
-    <child link = "base" />
+    <child link = "base_link" />
     <origin xyz="0.0 0.0 0.0" rpy="1.5708 0.0 1.5708" />
   </joint>

Commit message: Updated mount orientation + regenerated moveit

File: ur5_allegro.xacro (robot description, xacro)
@@ -19,10 +19,10 @@
     <parent link="tool0" />
     <child link = "mount_base" />
-    <origin xyz="0.0025 0.0 0.0" rpy="0.0 1.5708 0.0" />
+    <origin xyz="0.0025 0.0 0.0" rpy="0.0 0.0 0.0" />
   </joint>
   <joint name="mount_allegro" type="fixed">
     <parent link="mount_body" />
     <child link = "hand_root" />
-    <origin xyz="0.0 0.0 0.0375" rpy="0.0 0.0 2.356" />
+    <origin xyz="0.0 0.0 0.0375" rpy="0.0 0.0 -2.356" />
   </joint>
 </robot>

Commit message: Xacro file: repositioned the arm for metallic frame

File: ur5_allegro.xacro (robot description, xacro)
@@ -14,5 +14,5 @@
     <parent link="world" />
     <child link = "base_link" />
-    <origin xyz="0.0 0.0 0.0" rpy="1.5708 0.0 1.5708" />
+    <origin xyz="0.14 0.0 1.65" rpy="1.5708 0.0 1.5708" />
   </joint>
   <joint name="tool_mount" type="fixed">
