Commit message: Xacro: Base link position is adjusted

File: models/ur5_allegro.xacro (robot description, xacro)
@@ -14,5 +14,5 @@
     <parent link="world" />
     <child link = "base_link" />
-    <origin xyz="0.14 0.0 1.65" rpy="1.5708 0.0 1.5708" />
+    <origin xyz="0.145 0.0 1.656" rpy="1.5708 0.0 1.5708" />
   </joint>
   <joint name="tool_mount" type="fixed">

Commit message: Rotated the mount base

File: models/ur5_allegro.xacro (robot description, xacro)
@@ -24,5 +24,5 @@
     <parent link="mount_body" />
     <child link = "hand_root" />
-    <origin xyz="0.0 0.0 0.0375" rpy="0.0 0.0 -2.356" />
+    <origin xyz="0.0 0.0 0.0375" rpy="0.0 0.0 -0.79" />
   </joint>
 </robot>

Commit message: sep commit

File: models/ur5_allegro.xacro (robot description, xacro)
@@ -24,4 +24,5 @@
     <parent link="mount_body" />
     <child link = "hand_root" />
+    <!-- <origin xyz="0.0 0.0 0.0375" rpy="0.0 0.0 -2.356" /> -->
     <origin xyz="0.0 0.0 0.0375" rpy="0.0 0.0 -0.79" />
   </joint>

Commit message: oct2020

File: models/ur5_allegro.xacro (robot description, xacro)
@@ -2,6 +2,12 @@
 <!--- <robot xmlns:xacro="http://ros.org/wiki/xacro" name="ur5" >  -->
 <robot xmlns:xacro="http://ros.org/wiki/xacro" name="ur5_allegro" >
+  <xacro:arg name="optoforce" default="true"/>
   <!-- allegro -->
-  <xacro:include filename="$(find ur5_allegro_moveit)/models/allegro_optoforce_right.xacro" />
+  <xacro:if value="$(arg optoforce)">
+    <xacro:include filename="$(find ur5_allegro_moveit)/models/allegro_optoforce_right.xacro" />
+  </xacro:if>
+  <xacro:unless value="$(arg optoforce)">
+    <xacro:include filename="$(find allegro_hand_description)/allegro_hand_description_right.xacro" />
+  </xacro:unless>
   <!-- ur5 -->
   <xacro:include filename="$(find ur_description)/urdf/ur5.urdf.xacro" />
@@ -24,5 +30,4 @@
     <parent link="mount_body" />
     <child link = "hand_root" />
-    <!-- <origin xyz="0.0 0.0 0.0375" rpy="0.0 0.0 -2.356" /> -->
     <origin xyz="0.0 0.0 0.0375" rpy="0.0 0.0 -0.79" />
   </joint>
